Commit message: Thursday2

File: src/nexus_4wd_mecanum_description/urdf/rubot_mecanum.xacro (robot description, xacro)
@@ -350,5 +350,5 @@
   <joint name="joint_camera" type="fixed">
     <axis xyz="0 0 1" />
-    <origin xyz="0.25 0 0.025" rpy="0 0 0"/>
+    <origin xyz="0.16 0 0.08" rpy="0 0 0"/>
     <parent link="base_link"/>
     <child link="camera"/>
@@ -359,5 +359,5 @@
       <origin xyz="0 0 0.04" rpy="0 0 0" />
       <geometry>
-        <mesh filename="package://nexus_4wd_mecanum_description/meshes/X4.stl" scale="0.002 0.002 0.002"/>
+        <mesh filename="package://nexus_4wd_mecanum_description/meshes/X4.stl" scale="0.0015 0.0015 0.0015"/>
       </geometry>
       <material name="yellow"/>
@@ -380,10 +380,10 @@
   <joint name="scan_joint" type="fixed">
     <axis xyz="0 0 1" />
-    <origin xyz="0 0 0.15" rpy="0 0 0"/>
+    <origin xyz="0 0 0.09" rpy="0 0 0"/>
     <parent link="base_link"/>
     <child link="base_scan"/>
   </joint>
   <!-- Include controller plugin for Gazebo -->
-  <xacro:include filename="$(find nexus_4wd_mecanum_description)/urdf/nexus_4wd_mecanum.gazebo" />
+  <xacro:include filename="$(find nexus_4wd_mecanum_description)/urdf/rubot_mecanum.gazebo" />
   <!-- Include URM04 ultrasonic range finders -->
   <xacro:include filename="$(find nexus_4wd_mecanum_description)/urdf/urm04_sensor.xacro"/>

Commit message: Navigation

File: src/nexus_4wd_mecanum_description/urdf/rubot_mecanum.xacro (robot description, xacro)
@@ -350,5 +350,5 @@
   <joint name="joint_camera" type="fixed">
     <axis xyz="0 0 1" />
-    <origin xyz="0.16 0 0.08" rpy="0 0 0"/>
+    <origin xyz="0.16 0 0.05" rpy="0 0 0"/>
     <parent link="base_link"/>
     <child link="camera"/>
