Commit message: Added rubot model

File: src/robot_description/rubot_mecanum/urdf/rubot_mecanum.urdf (robot description, URDF)
Before this commit: robot prototip_2904, 18 links, 17 joints
Links:
- link Coberta_Link: geometry collision mesh filename=package://rubot_mecanum/meshes/Coberta_Link.STL; visual mesh filename=package://rubot_mecanum/meshes/Coberta_Link.STL
- link L1_Link: geometry collision mesh filename=package://rubot_mecanum/meshes/L1_Link.STL; visual mesh filename=package://rubot_mecanum/meshes/L1_Link.STL
- link L2_Link: geometry collision mesh filename=package://rubot_mecanum/meshes/L2_Link.STL; visual mesh filename=package://rubot_mecanum/meshes/L2_Link.STL
- link Lidar_Link: geometry collision mesh filename=package://rubot_mecanum/meshes/Lidar_Link.STL; visual mesh filename=package://rubot_mecanum/meshes/Lidar_Link.STL
- link ML1_Link: geometry collision mesh filename=package://rubot_mecanum/meshes/ML1_Link.STL; visual mesh filename=package://rubot_mecanum/meshes/ML1_Link.STL
- link ML2_Link: geometry collision mesh filename=package://rubot_mecanum/meshes/ML2_Link.STL; visual mesh filename=package://rubot_mecanum/meshes/ML2_Link.STL
- link MR1_Link: geometry collision mesh filename=package://rubot_mecanum/meshes/MR1_Link.STL; visual mesh filename=package://rubot_mecanum/meshes/MR1_Link.STL
- link MR2_Link: geometry collision mesh filename=package://rubot_mecanum/meshes/MR2_Link.STL; visual mesh filename=package://rubot_mecanum/meshes/MR2_Link.STL
- link R1_Link: geometry collision mesh filename=package://rubot_mecanum/meshes/R1_Link.STL; visual mesh filename=package://rubot_mecanum/meshes/R1_Link.STL
- link R2_Link: geometry collision mesh filename=package://rubot_mecanum/meshes/R2_Link.STL; visual mesh filename=package://rubot_mecanum/meshes/R2_Link.STL
- link SuportCentre1_Link: geometry collision mesh filename=package://rubot_mecanum/meshes/SuportCentre1_Link.STL; visual mesh filename=package://rubot_mecanum/meshes/SuportCentre1_Link.STL
- link SuportCentre2_Link: geometry collision mesh filename=package://rubot_mecanum/meshes/SuportCentre2_Link.STL; visual mesh filename=package://rubot_mecanum/meshes/SuportCentre2_Link.STL
- link SuportL1_Link: geometry collision mesh filename=package://rubot_mecanum/meshes/SuportL1_Link.STL; visual mesh filename=package://rubot_mecanum/meshes/SuportL1_Link.STL
- link SuportL2_Link: geometry collision mesh filename=package://rubot_mecanum/meshes/SuportL2_Link.STL; visual mesh filename=package://rubot_mecanum/meshes/SuportL2_Link.STL
- link SuportLidar_Link: geometry collision mesh filename=package://rubot_mecanum/meshes/SuportLidar_Link.STL; visual mesh filename=package://rubot_mecanum/meshes/SuportLidar_Link.STL
- link SuportR1_Link: geometry collision mesh filename=package://rubot_mecanum/meshes/SuportR1_Link.STL; visual mesh filename=package://rubot_mecanum/meshes/SuportR1_Link.STL
- link SuportR2_Link: geometry collision mesh filename=package://rubot_mecanum/meshes/SuportR2_Link.STL; visual mesh filename=package://rubot_mecanum/meshes/SuportR2_Link.STL
- link base_link: geometry collision mesh filename=package://rubot_mecanum/meshes/base_link.STL; visual mesh filename=package://rubot_mecanum/meshes/base_link.STL

Commit message: Added corrections to rubot

File: src/robot_description/rubot_mecanum/urdf/rubot_mecanum.urdf (robot description, URDF)
Before this commit: robot rubot_mecanum, 18 links, 17 joints
Links:
- added link base_footprint
Joints:
- added joint base_link_joint: type fixed, parent base_footprint, child base_link, origin xyz=0 0 0.05 rpy=0 0 0
