Commit message: Corrections in nexus model

File: src/robot_description/nexus_4wd_mecanum_description/urdf/test.urdf (robot description, URDF)
Before this commit: robot nexus, 16 links, 15 joints
Links:
- removed link base_scan
- removed link camera
- link base_link: geometry collision mesh filename=package://nexus_4wd_mecanum_description/meshes/nexus_base_l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 scale=0.001 0.001 0.001; visual mesh filename=package://nexus_4wd_mecanum_description/meshes/nexus_base_l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 scale=0.001 0.001 0.001
- link front_sensor: geometry visual mesh filename=package://nexus_4wd_mecanum_description/meshes/urm04.STL scale=0.001 0.001 0.001
- link left_sensor: geometry visual mesh filename=package://nexus_4wd_mecanum_description/meshes/urm04.STL scale=0.001 0.001 0.001
- link lower_left_wheel: geometry collision cylinder length=0.0505 radius=0.05; visual mesh filename=package://nexus_4wd_mecanum_description/meshes/mecanum_whee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 scale=0.001 0.001 0.001
- link lower_left_wheel_shaft: geometry collision mesh filename=package://nexus_4wd_mecanum_description/meshes/wheel_shaft.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 scale=0.001 0.001 0.001; visual mesh filename=package://nexus_4wd_mecanum_description/meshes/wheel_shaft.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 scale=0.001 0.001 0.001
- link lower_right_wheel: geometry collision cylinder length=0.0505 radius=0.05; visual mesh filename=package://nexus_4wd_mecanum_description/meshes/mecanum_whee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 scale=0.001 0.001 0.001
- link lower_right_wheel_shaft: geometry collision mesh filename=package://nexus_4wd_mecanum_description/meshes/wheel_shaft.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 scale=0.001 0.001 0.001; visual mesh filename=package://nexus_4wd_mecanum_description/meshes/wheel_shaft.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 scale=0.001 0.001 0.001
- link rear_sensor: geometry visual mesh filename=package://nexus_4wd_mecanum_description/meshes/urm04.STL scale=0.001 0.001 0.001
- link right_sensor: geometry visual mesh filename=package://nexus_4wd_mecanum_description/meshes/urm04.STL scale=0.001 0.001 0.001
- link upper_left_wheel: geometry collision cylinder length=0.0505 radius=0.05; visual mesh filename=package://nexus_4wd_mecanum_description/meshes/mecanum_whee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 scale=0.001 0.001 0.001
- link upper_left_wheel_shaft: geometry collision mesh filename=package://nexus_4wd_mecanum_description/meshes/wheel_shaft.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 scale=0.001 0.001 0.001; visual mesh filename=package://nexus_4wd_mecanum_description/meshes/wheel_shaft.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 scale=0.001 0.001 0.001
- link upper_right_wheel: geometry collision cylinder length=0.0505 radius=0.05; visual mesh filename=package://nexus_4wd_mecanum_description/meshes/mecanum_whee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 scale=0.001 0.001 0.001
- link upper_right_wheel_shaft: geometry collision mesh filename=package://nexus_4wd_mecanum_description/meshes/wheel_shaft.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 scale=0.001 0.001 0.001; visual mesh filename=package://nexus_4wd_mecanum_description/meshes/wheel_shaft.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 scale=0.001 0.001 0.001
Joints:
- removed joint joint_camera
- removed joint scan_joint
