Commit message: Corrections mecanum packages

File: src/robot_description/nexus_mecanum/urdf/nexus.urdf (robot description, URDF)
Before this commit: robot nexus, 16 links, 15 joints
Links:
- link base_link: geometry collision mesh filename=package://nexus_mecanum/meshes/nexus_base_link_collision.STL scale=0.001 0.001 0.001; visual mesh filename=package://nexus_mecanum/meshes/nexus_base_link.STL scale=0.001 0.001 0.001
- link base_scan: geometry collision cylinder length=0.01575 radius=0.0275; visual mesh filename=package://nexus_mecanum/meshes/X4.stl scale=0.0015 0.0015 0.0015
- link camera: geometry collision box size=0.075 0.075 0.025; visual mesh filename=package://nexus_mecanum/meshes/piCamera.stl scale=0.0025 0.0025 0.0025
- link front_sensor: geometry visual mesh filename=package://nexus_mecanum/meshes/urm04.STL scale=0.001 0.001 0.001
- link left_sensor: geometry visual mesh filename=package://nexus_mecanum/meshes/urm04.STL scale=0.001 0.001 0.001
- link lower_left_wheel: geometry collision cylinder length=0.0505 radius=0.05; visual mesh filename=package://nexus_mecanum/meshes/mecanum_wheel_right.STL scale=0.001 0.001 0.001
- link lower_left_wheel_shaft: geometry collision mesh filename=package://nexus_mecanum/meshes/wheel_shaft.STL scale=0.001 0.001 0.001; visual mesh filename=package://nexus_mecanum/meshes/wheel_shaft.STL scale=0.001 0.001 0.001
- link lower_right_wheel: geometry collision cylinder length=0.0505 radius=0.05; visual mesh filename=package://nexus_mecanum/meshes/mecanum_wheel_left.STL scale=0.001 0.001 0.001
- link lower_right_wheel_shaft: geometry collision mesh filename=package://nexus_mecanum/meshes/wheel_shaft.STL scale=0.001 0.001 0.001; visual mesh filename=package://nexus_mecanum/meshes/wheel_shaft.STL scale=0.001 0.001 0.001
- link rear_sensor: geometry visual mesh filename=package://nexus_mecanum/meshes/urm04.STL scale=0.001 0.001 0.001
- link right_sensor: geometry visual mesh filename=package://nexus_mecanum/meshes/urm04.STL scale=0.001 0.001 0.001
- link upper_left_wheel: geometry collision cylinder length=0.0505 radius=0.05; visual mesh filename=package://nexus_mecanum/meshes/mecanum_wheel_left.STL scale=0.001 0.001 0.001
- link upper_left_wheel_shaft: geometry collision mesh filename=package://nexus_mecanum/meshes/wheel_shaft.STL scale=0.001 0.001 0.001; visual mesh filename=package://nexus_mecanum/meshes/wheel_shaft.STL scale=0.001 0.001 0.001
- link upper_right_wheel: geometry collision cylinder length=0.0505 radius=0.05; visual mesh filename=package://nexus_mecanum/meshes/mecanum_wheel_right.STL scale=0.001 0.001 0.001
- link upper_right_wheel_shaft: geometry collision mesh filename=package://nexus_mecanum/meshes/wheel_shaft.STL scale=0.001 0.001 0.001; visual mesh filename=package://nexus_mecanum/meshes/wheel_shaft.STL scale=0.001 0.001 0.001

Commit message: nexus spawn

File: src/robot_description/nexus_mecanum/urdf/nexus.urdf (robot description, URDF)
Before this commit: robot nexus, 16 links, 15 joints
Joints:
- joint scan_joint: origin xyz=0 0 0.09 rpy=0 0 0 -> xyz=0 0 0.09 rpy=0 0 3.14
