Commit message: rubot model rviz

File: src/rubot_mecanum_description/urdf/rubot.urdf (robot description, URDF)
Before this commit: robot nexus, 8 links, 7 joints
Links:
- link base_scan: geometry collision cylinder length=0.01575 radius=0.0275; visual mesh filename=package://rubot_mecanum_description/meshes/rubot/lidar.stl scale=0.001 0.001 0.001
- link camera: geometry collision box size=0.075 0.075 0.025; visual mesh filename=package://rubot_mecanum_description/meshes/rubot/picam.stl scale=0.001 0.001 0.001
- link lower_right_wheel: geometry collision cylinder length=0.0505 radius=0.05; visual mesh filename=package://rubot_mecanum_description/meshes/rubot/wheel_righ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 scale=0.001 0.001 0.001
Joints:
- joint joint_camera: origin xyz=0.24 0.076 0.072 rpy=0 0 0 -> xyz=0 0 0 rpy=0 0 0
- joint lower_left_wheel_joint: origin xyz=0.046 0.181 -0.028 rpy=0 0 0 -> xyz=0 0 0 rpy=0 0 0
- joint lower_right_wheel_joint: origin xyz=0 0.042 0 rpy=0 0 0 -> xyz=0 0 0 rpy=0 0 0; parent lower_right_wheel_shaft -> base_link
- joint upper_right_wheel_joint: origin xyz=0.201 -0.031 -0.028 rpy=0 0 0 -> xyz=0 0 0 rpy=0 0 0

Commit message: rUBot model optimization

File: src/rubot_mecanum_description/urdf/rubot.urdf (robot description, URDF)
Before this commit: robot nexus, 8 links, 7 joints
Links:
- link base_link: mass 2.844 -> 10
Joints:
- joint joint_camera: origin xyz=0 0 0 rpy=0 0 0 -> xyz=0.236 0.076 0.072 rpy=0 0 0
- joint scan_joint: origin xyz=0 0 0 rpy=0 0 0 -> xyz=0.111 0.076 0.124 rpy=0 0 0

Commit message: Freecad model shift

File: src/rubot_mecanum_description/urdf/rubot.urdf (robot description, URDF)
Before this commit: robot nexus, 8 links, 7 joints
Links:
- link lower_left_wheel: geometry collision mesh filename=package://rubot_mecanum_description/meshes/rubot/wheel_left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 scale=0.001 0.001 0.001; visual mesh filename=package://rubot_mecanum_description/meshes/rubot/wheel_left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 scale=0.001 0.001 0.001
- link lower_right_wheel: geometry collision mesh filename=package://rubot_mecanum_description/meshes/rubot/wheel_righ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 scale=0.001 0.001 0.001; visual mesh filename=package://rubot_mecanum_description/meshes/rubot/wheel_righ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 scale=0.001 0.001 0.001
- link upper_left_wheel: geometry collision mesh filename=package://rubot_mecanum_description/meshes/rubot/wheel_left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 scale=0.001 0.001 0.001; visual mesh filename=package://rubot_mecanum_description/meshes/rubot/wheel_left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 scale=0.001 0.001 0.001
- link upper_right_wheel: geometry collision mesh filename=package://rubot_mecanum_description/meshes/rubot/wheel_righ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 scale=0.001 0.001 0.001; visual mesh filename=package://rubot_mecanum_description/meshes/rubot/wheel_righ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 scale=0.001 0.001 0.001
Joints:
- joint base_link_joint: origin xyz=0 0 0.05 rpy=0 0 0 -> xyz=0 0 0 rpy=0 0 0
- joint joint_camera: origin xyz=0.236 0.076 0.072 rpy=0 0 0 -> xyz=0.236 0.076 0.1 rpy=0 0 0
- joint scan_joint: origin xyz=0.111 0.076 0.124 rpy=0 0 0 -> xyz=0.111 0.076 0.152 rpy=0 0 0

Commit message: model shift

File: src/rubot_mecanum_description/urdf/rubot.urdf (robot description, URDF)
Before this commit: robot nexus, 8 links, 7 joints
Links:
- link base_link: geometry collision box size=0.1 0.1 0.35; visual mesh filename=package://rubot_mecanum_description/meshes/rubot/base_link.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 scale=0.001 0.001 0.001
Joints:
- joint joint_camera: origin xyz=0.236 0.076 0.1 rpy=0 0 0 -> xyz=0.236 0.076 0.072 rpy=0 0 0
- joint scan_joint: origin xyz=0.111 0.076 0.152 rpy=0 0 0 -> xyz=0.111 0.076 0.124 rpy=0 0 0
